File: Project_Tsukuyomi (JapanOpen)/Hardware/KiCad/CAM/CAM.kicad_sch (KiCad schematic)
At the start: 29 parts, among them J1 Conn_01x04_Socket, J2 Conn_01x04_Socket, J3 Conn_01x04_Socket, J4 Conn_01x04_Socket, J5 Conn_01x04_Socket, J6 Conn_01x04_Socket, J7 Conn_01x04_Socket, U1 Teensy4.0, U2 AZ1084-5.0, U3 TSSP58P38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

Commit message: KiCad変更
ごめんさい。溜めました
Parts:
- C1: renamed from C3; footprint (none) -> Capacitor_THT:C_Disc_D3.0mm_W1.6mm_P2.50mm
- C2: renamed from C4; footprint (none) -> Capacitor_THT:C_Disc_D3.0mm_W1.6mm_P2.50mm
- C3: renamed from C5; footprint (none) -> Capacitor_THT:C_Disc_D3.0mm_W1.6mm_P2.50mm
- C4: renamed from C6; footprint (none) -> Capacitor_THT:C_Disc_D3.0mm_W1.6mm_P2.50mm
- C5: renamed from C7; footprint (none) -> Capacitor_THT:C_Disc_D3.0mm_W1.6mm_P2.50mm
- C6: renamed from C8; footprint (none) -> Capacitor_THT:C_Disc_D3.0mm_W1.6mm_P2.50mm
- C7: renamed from C1; footprint (none) -> Capacitor_THT:CP_Radial_D4.0mm_P2.00mm
- C8: renamed from C2; footprint (none) -> Capacitor_THT:C_Disc_D3.0mm_W1.6mm_P2.50mm
- J1, J2, J3, J4, J5, J6, J7: footprint (none) -> Connector_JST:JST_XH_B4B-XH-A_1x04_P2.50mm_Vertical
- R1, R2, R3, R4, R5, R6: footprint (none) -> Resistor_THT:R_Axial_DIN0204_L3.6mm_D1.6mm_P5.08mm_Horizontal
- U7: renamed from U2; footprint (none) -> Package_TO_SOT_SMD:TO-252-2
- U8: renamed from U1; footprint (none) -> Teensy_Breakout:Teensy_Brakeout
- renumbered U3 to U1, U4 to U2, U5 to U3, U6 to U4, U7 to U5, U8 to U6
