File: Project_Tsukuyomi (JapanOpen)/Hardware/KiCad/Line/Line.kicad_sch (KiCad schematic)
At the start: 190 parts, among them J1 USB_C_Receptacle_USB2.0, J2 Conn_01x04_Socket, Q1 Q_Photo_NPN, Q10 Q_Photo_NPN, Q11 Q_Photo_NPN, Q12 Q_Photo_NPN, Q13 Q_Photo_NPN, Q14 Q_Photo_NPN, Q15 Q_Photo_NPN, Q16 Q_Photo_NPN, Q17 Q_Photo_NPN, Q18 Q_Photo_NPN, Q19 Q_Photo_NPN, Q2 Q_Photo_NPN, Q20 Q_Photo_NPN, Q21 Q_Photo_NPN, Q22 Q_Photo_NPN, Q23 Q_Photo_NPN, Q24 Q_Photo_NPN, Q25 Q_Photo_NPN, Q26 Q_Photo_NPN, Q27 Q_Photo_NPN, Q28 Q_Photo_NPN, Q29 Q_Photo_NPN, Q3 Q_Photo_NPN, Q30 Q_Photo_NPN, Q31 Q_Photo_NPN, Q32 Q_Photo_NPN, Q33 Q_Photo_NPN, Q34 Q_Photo_NPN, Q35 Q_Photo_NPN, Q36 Q_Photo_NPN, Q37 Q_Photo_NPN, Q38 Q_Photo_NPN, Q39 Q_Photo_NPN, Q4 Q_Photo_NPN, Q40 Q_Photo_NPN, Q41 Q_Photo_NPN, Q42 Q_Photo_NPN, Q43 Q_Photo_NPN, Q44 Q_Photo_NPN, Q45 Q_Photo_NPN, Q46 Q_Photo_NPN, Q47 Q_Photo_NPN, Q48 Q_Photo_NPN, Q49 Q_Photo_NPN, Q5 Q_Photo_NPN, Q50 Q_Photo_NPN, Q51 Q_Photo_NPN, Q52 Q_Photo_NPN, Q53 Q_Photo_NPN, Q54 Q_Photo_NPN, Q55 Q_Photo_NPN, Q56 Q_Photo_NPN, Q57 Q_Photo_NPN, Q58 Q_Photo_NPN, Q59 Q_Photo_NPN, Q6 Q_Photo_NPN, Q60 Q_Photo_NPN, Q61 Q_Photo_NPN, Q62 Q_Photo_NPN, Q63 Q_Photo_NPN, Q64 Q_Photo_NPN, Q7 Q_Photo_NPN, Q8 Q_Photo_NPN, Q9 Q_Photo_NPN, SW1 SW_Push, SW2 SW_Push, U1 W25Q128JVS, U2 RP2040, U3 CD74HC4067SM, U4 CD74HC4067SM, U5 AZ1084-3.3, U6 AZ1084-5.0, Y1 Crystal_GND24

Commit message: KiCad変更
ごめんさい。溜めました
Parts:
- removed D17, D18, D25, D26, D33, D34, D41, D42, D49, D50, D57, D58: WS2812B, LED_SMD:LED_WS2812B_PLCC4_5.0x5.0mm_P3.2mm, symbol LED:WS2812B
- added D11, D12, D13, D14, D15, D16, D3, D4, D5, D6, D7, D8: WS2812B, LED_SMD:LED_WS2812B-2020_PLCC4_2.0x2.0mm, symbol LED:WS2812B
- C1: renamed from C12; footprint (none) -> Capacitor_SMD:C_1210_3225Metric
- C10: renamed from C8; footprint (none) -> Capacitor_SMD:C_0402_1005Metric; LCSC (none) -> C1525
- C11: renamed from C9; footprint (none) -> Capacitor_SMD:C_0402_1005Metric; LCSC (none) -> C1525
- C12: renamed from C3; footprint (none) -> Capacitor_SMD:C_0402_1005Metric; LCSC (none) -> C1525
- C13: renamed from C4; footprint (none) -> Capacitor_SMD:C_0402_1005Metric; LCSC (none) -> C1525
- C2: renamed from C13; footprint (none) -> Capacitor_SMD:C_0402_1005Metric; LCSC (none) -> C1525
- C3: renamed from C10; footprint (none) -> Capacitor_SMD:C_0402_1005Metric
- C4: renamed from C1; footprint (none) -> Capacitor_SMD:C_0402_1005Metric; LCSC (none) -> C1557
- C5: renamed from C2; footprint (none) -> Capacitor_SMD:C_0402_1005Metric; LCSC (none) -> C1557
- C6: renamed from C11; footprint (none) -> Capacitor_SMD:C_0402_1005Metric; LCSC (none) -> C1525
- C7: renamed from C5; footprint (none) -> Capacitor_SMD:C_0402_1005Metric; LCSC (none) -> C1525
- C8: renamed from C6; footprint (none) -> Capacitor_SMD:C_0402_1005Metric; LCSC (none) -> C1525
- C9: renamed from C7; footprint (none) -> Capacitor_SMD:C_0402_1005Metric; LCSC (none) -> C1525
- D1, D10, D19, D20, D21, D22, D23, D24, D27, D28, D29, D30, D31, D32, D35, D36, D37, D38, D39, D40, D43, D44, D45, D46, D47, D48, D51, D52, D53, D54, D55, D56, D59, D60, D61, D62, D63, D64: footprint LED_SMD:LED_WS2812B_PLCC4_5.0x5.0mm_P3.2mm -> LED_SMD:LED_WS2812B-2020_PLCC4_2.0x2.0mm; LCSC (none) -> C965555
- D17: renamed from D3; footprint LED_SMD:LED_WS2812B_PLCC4_5.0x5.0mm_P3.2mm -> LED_SMD:LED_WS2812B-2020_PLCC4_2.0x2.0mm; LCSC (none) -> C965555
- D18: renamed from D11; footprint LED_SMD:LED_WS2812B_PLCC4_5.0x5.0mm_P3.2mm -> LED_SMD:LED_WS2812B-2020_PLCC4_2.0x2.0mm; LCSC (none) -> C965555
- D2: renamed from D9; footprint LED_SMD:LED_WS2812B_PLCC4_5.0x5.0mm_P3.2mm -> LED_SMD:LED_WS2812B-2020_PLCC4_2.0x2.0mm; LCSC (none) -> C965555
- D25: renamed from D4; footprint LED_SMD:LED_WS2812B_PLCC4_5.0x5.0mm_P3.2mm -> LED_SMD:LED_WS2812B-2020_PLCC4_2.0x2.0mm; LCSC (none) -> C965555
- D26: renamed from D12; footprint LED_SMD:LED_WS2812B_PLCC4_5.0x5.0mm_P3.2mm -> LED_SMD:LED_WS2812B-2020_PLCC4_2.0x2.0mm; LCSC (none) -> C965555
- D33: renamed from D5; footprint LED_SMD:LED_WS2812B_PLCC4_5.0x5.0mm_P3.2mm -> LED_SMD:LED_WS2812B-2020_PLCC4_2.0x2.0mm; LCSC (none) -> C965555
- D34: renamed from D13; footprint LED_SMD:LED_WS2812B_PLCC4_5.0x5.0mm_P3.2mm -> LED_SMD:LED_WS2812B-2020_PLCC4_2.0x2.0mm; LCSC (none) -> C965555
- D41: renamed from D6; footprint LED_SMD:LED_WS2812B_PLCC4_5.0x5.0mm_P3.2mm -> LED_SMD:LED_WS2812B-2020_PLCC4_2.0x2.0mm; LCSC (none) -> C965555
- D42: renamed from D14; footprint LED_SMD:LED_WS2812B_PLCC4_5.0x5.0mm_P3.2mm -> LED_SMD:LED_WS2812B-2020_PLCC4_2.0x2.0mm; LCSC (none) -> C965555
- D49: renamed from D7; footprint LED_SMD:LED_WS2812B_PLCC4_5.0x5.0mm_P3.2mm -> LED_SMD:LED_WS2812B-2020_PLCC4_2.0x2.0mm; LCSC (none) -> C965555
- D50: renamed from D15; footprint LED_SMD:LED_WS2812B_PLCC4_5.0x5.0mm_P3.2mm -> LED_SMD:LED_WS2812B-2020_PLCC4_2.0x2.0mm; LCSC (none) -> C965555
- D57: renamed from D8; footprint LED_SMD:LED_WS2812B_PLCC4_5.0x5.0mm_P3.2mm -> LED_SMD:LED_WS2812B-2020_PLCC4_2.0x2.0mm; LCSC (none) -> C965555
- D58: renamed from D16; footprint LED_SMD:LED_WS2812B_PLCC4_5.0x5.0mm_P3.2mm -> LED_SMD:LED_WS2812B-2020_PLCC4_2.0x2.0mm; LCSC (none) -> C965555
- D9: renamed from D2; footprint LED_SMD:LED_WS2812B_PLCC4_5.0x5.0mm_P3.2mm -> LED_SMD:LED_WS2812B-2020_PLCC4_2.0x2.0mm; LCSC (none) -> C965555
- J1: renamed from J2; footprint (none) -> Connector_JST:JST_XH_B4B-XH-A_1x04_P2.50mm_Vertical
- J2: renamed from J1; footprint (none) -> Connector_USB:USB_C_Receptacle_GCT_USB4105-xx-A_16P_TopMnt_Horizontal; LCSC (none) -> C136423
- Q1: renamed from Q31; footprint (none) -> NJL7502R:NJL7502
- Q10: renamed from Q3; footprint (none) -> NJL7502R:NJL7502
- Q11: renamed from Q38; footprint (none) -> NJL7502R:NJL7502
- Q12: renamed from Q4; footprint (none) -> NJL7502R:NJL7502
- Q13: renamed from Q39; footprint (none) -> NJL7502R:NJL7502
- Q14: renamed from Q5; footprint (none) -> NJL7502R:NJL7502
- Q15: renamed from Q40; footprint (none) -> NJL7502R:NJL7502
- Q16: renamed from Q6; footprint (none) -> NJL7502R:NJL7502
- Q17: renamed from Q41; footprint (none) -> NJL7502R:NJL7502
- Q18: renamed from Q7; footprint (none) -> NJL7502R:NJL7502
- Q19: renamed from Q42; footprint (none) -> NJL7502R:NJL7502
- Q2: renamed from Q33; footprint (none) -> NJL7502R:NJL7502
- Q20: renamed from Q8; footprint (none) -> NJL7502R:NJL7502
- Q21: renamed from Q43; footprint (none) -> NJL7502R:NJL7502
- Q22: renamed from Q9; footprint (none) -> NJL7502R:NJL7502
- Q23: renamed from Q44; footprint (none) -> NJL7502R:NJL7502
- Q24: renamed from Q10; footprint (none) -> NJL7502R:NJL7502
- Q25: renamed from Q45; footprint (none) -> NJL7502R:NJL7502
- Q26: renamed from Q11; footprint (none) -> NJL7502R:NJL7502
- Q27: renamed from Q46; footprint (none) -> NJL7502R:NJL7502
- Q28: renamed from Q12; footprint (none) -> NJL7502R:NJL7502
- Q29: renamed from Q47; footprint (none) -> NJL7502R:NJL7502
- Q3: renamed from Q32; footprint (none) -> NJL7502R:NJL7502
- Q30: renamed from Q13; footprint (none) -> NJL7502R:NJL7502
- Q31: renamed from Q48; footprint (none) -> NJL7502R:NJL7502
- Q32: renamed from Q14; footprint (none) -> NJL7502R:NJL7502
- Q33: renamed from Q49; footprint (none) -> NJL7502R:NJL7502
- Q34: renamed from Q15; footprint (none) -> NJL7502R:NJL7502
- Q35: renamed from Q50; footprint (none) -> NJL7502R:NJL7502
- Q36: renamed from Q16; footprint (none) -> NJL7502R:NJL7502
- Q37: renamed from Q51; footprint (none) -> NJL7502R:NJL7502
- Q38: renamed from Q17; footprint (none) -> NJL7502R:NJL7502
- Q39: renamed from Q52; footprint (none) -> NJL7502R:NJL7502
- Q4: renamed from Q34; footprint (none) -> NJL7502R:NJL7502
- Q40: renamed from Q18; footprint (none) -> NJL7502R:NJL7502
- Q41: renamed from Q53; footprint (none) -> NJL7502R:NJL7502
- Q42: renamed from Q19; footprint (none) -> NJL7502R:NJL7502
- Q43: renamed from Q54; footprint (none) -> NJL7502R:NJL7502
- Q44: renamed from Q20; footprint (none) -> NJL7502R:NJL7502
- Q45: renamed from Q55; footprint (none) -> NJL7502R:NJL7502
- Q46: renamed from Q21; footprint (none) -> NJL7502R:NJL7502
- Q47: renamed from Q56; footprint (none) -> NJL7502R:NJL7502
- Q48: renamed from Q22; footprint (none) -> NJL7502R:NJL7502
- Q49: renamed from Q57; footprint (none) -> NJL7502R:NJL7502
- Q5: renamed from Q35; footprint (none) -> NJL7502R:NJL7502
- Q50: renamed from Q23; footprint (none) -> NJL7502R:NJL7502
- Q51: renamed from Q58; footprint (none) -> NJL7502R:NJL7502
- Q52: renamed from Q24; footprint (none) -> NJL7502R:NJL7502
- Q53: renamed from Q59; footprint (none) -> NJL7502R:NJL7502
- Q54: renamed from Q25; footprint (none) -> NJL7502R:NJL7502
- Q55: renamed from Q60; footprint (none) -> NJL7502R:NJL7502
- Q56: renamed from Q26; footprint (none) -> NJL7502R:NJL7502
- Q57: renamed from Q61; footprint (none) -> NJL7502R:NJL7502
- Q58: renamed from Q27; footprint (none) -> NJL7502R:NJL7502
- Q59: renamed from Q62; footprint (none) -> NJL7502R:NJL7502
- Q6: renamed from Q1; footprint (none) -> NJL7502R:NJL7502
- Q60: renamed from Q28; footprint (none) -> NJL7502R:NJL7502
- Q61: renamed from Q63; footprint (none) -> NJL7502R:NJL7502
- Q62: renamed from Q29; footprint (none) -> NJL7502R:NJL7502
- Q63: renamed from Q64; footprint (none) -> NJL7502R:NJL7502
- Q64: renamed from Q30; footprint (none) -> NJL7502R:NJL7502
- Q7: renamed from Q36; footprint (none) -> NJL7502R:NJL7502
- Q8: renamed from Q2; footprint (none) -> NJL7502R:NJL7502
- Q9: renamed from Q37; footprint (none) -> NJL7502R:NJL7502
- R1: renamed from R18; footprint (none) -> Resistor_SMD:R_0603_1608Metric
- R10: renamed from R6; footprint (none) -> Resistor_SMD:R_0603_1608Metric
- R11: renamed from R24; footprint (none) -> Resistor_SMD:R_0603_1608Metric
- R12: renamed from R7; footprint (none) -> Resistor_SMD:R_0603_1608Metric
- R13: renamed from R25; footprint (none) -> Resistor_SMD:R_0603_1608Metric
- R14: renamed from R8; footprint (none) -> Resistor_SMD:R_0603_1608Metric
- R15: renamed from R26; footprint (none) -> Resistor_SMD:R_0603_1608Metric
- R16: renamed from R9; footprint (none) -> Resistor_SMD:R_0603_1608Metric
- R17: renamed from R27; footprint (none) -> Resistor_SMD:R_0603_1608Metric
- R18: renamed from R10; footprint (none) -> Resistor_SMD:R_0603_1608Metric
- R19: renamed from R28; footprint (none) -> Resistor_SMD:R_0603_1608Metric
- R2: renamed from R19; footprint (none) -> Resistor_SMD:R_0603_1608Metric
- R20: renamed from R11; footprint (none) -> Resistor_SMD:R_0603_1608Metric
- R21: renamed from R29; footprint (none) -> Resistor_SMD:R_0603_1608Metric
- R22: renamed from R12; footprint (none) -> Resistor_SMD:R_0603_1608Metric
- R23: renamed from R30; footprint (none) -> Resistor_SMD:R_0603_1608Metric
- R24: renamed from R13; footprint (none) -> Resistor_SMD:R_0603_1608Metric
- R25: renamed from R38; footprint (none) -> Resistor_SMD:R_0402_1005Metric; LCSC (none) -> C25100
- R26: renamed from R35; footprint (none) -> Resistor_SMD:R_0402_1005Metric; LCSC (none) -> C25905
- R27: renamed from R36; footprint (none) -> Resistor_SMD:R_0402_1005Metric; LCSC (none) -> C25905
- R28: renamed from R31; footprint (none) -> Resistor_SMD:R_0603_1608Metric
- R29: renamed from R14; footprint (none) -> Resistor_SMD:R_0603_1608Metric
- R3: renamed from R20; footprint (none) -> Resistor_SMD:R_0603_1608Metric
- R30: renamed from R1; footprint (none) -> Resistor_SMD:R_0402_1005Metric; LCSC (none) -> C11702
- R31: renamed from R37; footprint (none) -> Resistor_SMD:R_0402_1005Metric; LCSC (none) -> C25100
- R32: renamed from R2; footprint (none) -> Resistor_SMD:R_0402_1005Metric; LCSC (none) -> C11702
- R33: renamed from R32; footprint (none) -> Resistor_SMD:R_0603_1608Metric
- R34: renamed from R15; footprint (none) -> Resistor_SMD:R_0603_1608Metric
- R35: renamed from R33; footprint (none) -> Resistor_SMD:R_0603_1608Metric
- R36: renamed from R16; footprint (none) -> Resistor_SMD:R_0603_1608Metric
- R37: renamed from R34; footprint (none) -> Resistor_SMD:R_0603_1608Metric
- R38: renamed from R17; footprint (none) -> Resistor_SMD:R_0603_1608Metric
- R4: renamed from R3; footprint (none) -> Resistor_SMD:R_0603_1608Metric
- R5: renamed from R21; footprint (none) -> Resistor_SMD:R_0603_1608Metric
- R6: renamed from R4; footprint (none) -> Resistor_SMD:R_0603_1608Metric
- R7: renamed from R22; footprint (none) -> Resistor_SMD:R_0603_1608Metric
- R8: renamed from R5; footprint (none) -> Resistor_SMD:R_0603_1608Metric
- R9: renamed from R23; footprint (none) -> Resistor_SMD:R_0603_1608Metric
- SW1: renamed from SW2; footprint (none) -> Button_Switch_SMD:SW_SPST_B3U-1000P
- SW2: renamed from SW1; footprint (none) -> Button_Switch_SMD:SW_SPST_B3U-1000P
- U1: renamed from U6; footprint (none) -> Package_TO_SOT_SMD:TO-252-2
- U2: renamed from U3; LCSC (none) -> C98457
- U3: renamed from U4; LCSC (none) -> C98457
- U4: renamed from U5; footprint (none) -> Package_TO_SOT_SMD:SOT-23-3
- U5: renamed from U1; LCSC (none) -> C97521
- U6: renamed from U2; LCSC (none) -> RP2040
- Y1: footprint (none) -> Crystal:Crystal_SMD_3225-4Pin_3.2x2.5mm; LCSC (none) -> C7294610
Connections:
- net +5V: now also D11.1 (VDD), D12.1 (VDD), D13.1 (VDD), D14.1 (VDD), D15.1 (VDD), D16.1 (VDD), D3.1 (VDD), D4.1 (VDD), D5.1 (VDD), D6.1 (VDD), D7.1 (VDD), D8.1 (VDD)
- net B: now also D3.4 (DIN)
- net C: now also D59.2 (DOUT), D4.4 (DIN); no longer D31.2 (DOUT)
- net D: now also D60.2 (DOUT), D5.4 (DIN); no longer D32.2 (DOUT)
- net E: now also D6.4 (DIN)
- net F: now also D7.4 (DIN); no longer D35.4 (DIN)
- net G: now also D8.4 (DIN); no longer D36.4 (DIN)
- net GND: now also D11.3 (VSS), D12.3 (VSS), D13.3 (VSS), D14.3 (VSS), D15.3 (VSS), D16.3 (VSS), D3.3 (VSS), D4.3 (VSS), D5.3 (VSS), D6.3 (VSS), D7.3 (VSS), D8.3 (VSS)
- net at D46.2 (DOUT): now also D54.4 (DIN)
- net at D46.4 (DIN): now also D38.2 (DOUT)
- net at D48.2 (DOUT): now also D56.4 (DIN); no longer D52.4 (DIN)
- net at D48.4 (DIN): now also D40.2 (DOUT); no longer D44.2 (DOUT)
- net at D23.2 (DOUT): now also D31.4 (DIN)
- net at D21.2 (DOUT): now also D29.4 (DIN); no longer D23.4 (DIN)
- net at D22.4 (DIN): now also D14.2 (DOUT); no longer D20.2 (DOUT)
- net at D20.4 (DIN): now also D12.2 (DOUT)
- net at D62.4 (DIN): now also D54.2 (DOUT)
- net at D36.2 (DOUT): now also D44.4 (DIN); no longer D40.4 (DIN)
- net at D64.4 (DIN): now also D56.2 (DOUT); no longer D60.2 (DOUT)
- net at D60.4 (DIN): now also D52.2 (DOUT); no longer D56.2 (DOUT)
- net at D38.4 (DIN): now also D30.2 (DOUT)
- net at D21.4 (DIN): now also D13.2 (DOUT); no longer D19.2 (DOUT)
- net at D19.4 (DIN): now also D11.2 (DOUT)
- net at D29.2 (DOUT): now also D37.4 (DIN); no longer D31.4 (DIN)
- net at D27.2 (DOUT): now also D35.4 (DIN); no longer D29.4 (DIN)
- net at D53.4 (DIN): now also D45.2 (DOUT)
- net at D45.4 (DIN): now also D37.2 (DOUT)
- net at D39.4 (DIN): now also D31.2 (DOUT); no longer D35.2 (DOUT)
- net at D24.2 (DOUT): now also D32.4 (DIN)
- net at D24.4 (DIN): now also D16.2 (DOUT); no longer D22.2 (DOUT)
- net at D61.4 (DIN): now also D53.2 (DOUT)
- net at D28.2 (DOUT): now also D36.4 (DIN); no longer D30.4 (DIN)
- net at D63.4 (DIN): now also D55.2 (DOUT); no longer D59.2 (DOUT)
- net at D59.4 (DIN): now also D51.2 (DOUT); no longer D55.2 (DOUT)
- net at D55.4 (DIN): now also D47.2 (DOUT); no longer D51.2 (DOUT)
- net at D47.4 (DIN): now also D39.2 (DOUT); no longer D43.2 (DOUT)
- net at D43.4 (DIN): now also D35.2 (DOUT); no longer D39.2 (DOUT)
- net at D51.4 (DIN): now also D43.2 (DOUT); no longer D47.2 (DOUT)
- net at D28.4 (DIN): now also D20.2 (DOUT)
- net at D27.4 (DIN): now also D19.2 (DOUT)
- new net: D16.4 (DIN), D8.2 (DOUT)
- new net: D14.4 (DIN), D6.2 (DOUT)
- new net: D13.4 (DIN), D5.2 (DOUT)
- new net: D15.2 (DOUT), D23.4 (DIN)
- new net: D15.4 (DIN), D7.2 (DOUT)
- new net: D11.4 (DIN), D3.2 (DOUT)
- new net: D44.2 (DOUT), D52.4 (DIN)
- new net: D22.2 (DOUT), D30.4 (DIN)
- new net: D12.4 (DIN), D4.2 (DOUT)
- new net: D32.2 (DOUT), D40.4 (DIN)
- no-connect marks 6 -> 22
Other:
- moved on the sheet: D1, D10, D17, D18, D2, D25, D26, D33, D34, D41, D42, D49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
