File: Project_Tsukuyomi (JapanOpen)/Hardware/KiCad/MD/MD.kicad_pcb (KiCad board)
At the start: 2 copper layers, 38 x 37.2 mm, 38 parts, among them J1 USB_C_Receptacle_USB2.0, J2 Conn_01x08_Socket, J3 Conn_01x08_Socket, J4 Conn_01x02_Socket, J5 Conn_01x02_Socket, J6 Conn_01x02_Socket, J7 Conn_01x02_Socket, SW1 SW_Push, SW2 SW_Push, U1 W25Q128JVS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

Commit message: KiCad変更
ごめんさい。溜めました
Parts:
- removed C8: 0.1μ, Capacitor_SMD:C_0402_1005Metric
- added C10: 0.1μ, Capacitor_SMD:C_1210_3225Metric_Pad1.33x2.70mm_HandSolder, F.Cu at (166.1, 78.2)
- added C11: 0.1μ, Capacitor_SMD:C_0402_1005Metric, F.Cu at (164.6, 90.7)
- added REF**: TestPoint_Keystone_5000-5004_Miniature, TestPoint:TestPoint_Keystone_5000-5004_Miniature, F.Cu at (148.7, 74.9)
- added REF**: TestPoint_Keystone_5000-5004_Miniature, TestPoint:TestPoint_Keystone_5000-5004_Miniature, F.Cu at (154.8, 74.9)
- added REF**: MountingHole_2.1mm, MountingHole:MountingHole_2.1mm, F.Cu at (135.3, 99.0)
- added REF**: TestPoint_Keystone_5000-5004_Miniature, TestPoint:TestPoint_Keystone_5000-5004_Miniature, F.Cu at (161.0, 74.8)
- added REF**: TestPoint_Keystone_5000-5004_Miniature, TestPoint:TestPoint_Keystone_5000-5004_Miniature, F.Cu at (142.1, 74.9)
- added U7: AZ1084-3.3, Package_TO_SOT_SMD:TO-252-2, F.Cu at (164.6, 85.5)
- Y1: footprint Crystal:Crystal_SMD_2016-4Pin_2.0x1.6mm -> Crystal:Crystal_SMD_2520-4Pin_2.5x2.0mm
- moved SW1 19.6 mm to (156.5, 83.1), turned to -90 degrees
- moved U5 19.2 mm to (148.7, 75.2)
- moved U3 18.9 mm to (142.1, 75.2)
- moved SW2 11.2 mm to (159.5, 83.1), turned to -90 degrees
- moved R5 10.2 mm to (160.0, 80.1)
- moved D2 9.43 mm to (137.4, 77.5), turned to -90 degrees
- moved R8 9.33 mm to (137.4, 80.1), turned to 90 degrees
- moved U1 8.21 mm to (155.3, 89.2), turned to 180 degrees
- moved D3 7.75 mm to (138.6, 77.5), turned to -90 degrees
- moved R9 7.64 mm to (138.6, 80.1), turned to 90 degrees
- moved C1 7.09 mm to (151.6, 80.8), turned to -90 degrees
- moved Y1 6.35 mm to (149.1, 80.8)
- moved R2 5.81 mm to (135.6, 95.9), turned to 180 degrees
- moved R1 5.56 mm to (135.6, 95.0), turned to 180 degrees
- moved C2 5.14 mm to (146.6, 80.0)
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- renumbered R12 to R3, R13 to R4
Routing:
- net +12V: track 0.00 -> 295.8 mm, vias 0 -> 22
- net +3.3V: track 8.38 -> 106.2 mm, vias 0 -> 4
- net GND: track 3.58 -> 61.9 mm, vias 1 -> 57
- net /MDRX: track 0.00 -> 31.4 mm, vias 0 -> 1
- net /RUN: track 2.53 -> 31.2 mm, vias 0 -> 2
- net /BLDC2: track 0.00 -> 24.5 mm, vias 0 -> 1
- net /MDTX: track 0.00 -> 24.5 mm, vias 0 -> 1
- net /BLDC1: track 0.00 -> 24.0 mm, vias 0 -> 1
- net /IN3B: track 0.00 -> 21.7 mm, vias 0 -> 2
- net /IN3A: track 0.00 -> 21.1 mm, vias 0 -> 2
- net /IN1B: track 0.00 -> 20.6 mm, vias 0 -> 2
- net /IN4A: track 0.00 -> 19.4 mm, vias 0 -> 2
- net /IN4B: track 0.00 -> 17.8 mm, vias 0 -> 2
- net +1V1: track 0.00 -> 15.8 mm
- net Net-(U1-~{CS}): track 15.5 -> 30.3 mm
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- added copper zone on B.Cu, net GND
- added copper zone on F.Cu, net GND
