File: Project_Tsukuyomi (JapanOpen)/Hardware/KiCad/MD/MD.kicad_sch (KiCad schematic)
At the start: 41 parts, among them J2 Conn_01x08_Socket, J3 Conn_01x08_Socket, J4 Conn_01x02_Socket, J5 Conn_01x02_Socket, J6 Conn_01x02_Socket, J7 Conn_01x02_Socket, J7 USB_C_Receptacle_USB2.0, SW3 SW_Push, SW4 SW_Push, U1 RP2040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

Commit message: KiCad変更
ごめんさい。溜めました
Parts:
- added C10, C11: 0.1μ, Capacitor_SMD:C_0402_1005Metric, symbol Device:C
- added U7: AZ1084-3.3, Package_TO_SOT_SMD:TO-252-2, symbol Regulator_Linear:AZ1084-3.3
- C12, C13, C3, C6, C7, C8, C9: LCSC (none) -> C1525
- C4, C5: LCSC (none) -> C1557
- J4, J5, J6, J7: footprint Connector_JST:JST_XH_S2B-XH-A_1x02_P2.50mm_Horizontal -> Connector_JST:JST_XH_B2B-XH-A_1x02_P2.50mm_Vertical
- J7: LCSC (none) -> C136423
- R10, R11, R4, R6: LCSC (none) -> C11702
- R12: LCSC (none) -> C25076
- R17, R18: LCSC (none) -> C25905
- R19, R20: LCSC (none) -> C25100
- U1: LCSC (none) -> C2040
- U4: LCSC (none) -> C97521
- Y1: LCSC (none) -> C7294610
Connections:
- net +12V: now also C10.2, U7.3 (VI)
- net +3.3V: now also C11.2, U7.2 (VO)
- net GND: now also C10.1, C11.1, U7.1 (GND)
