File: Project_Tsukuyomi (JapanOpen)/Hardware/KiCad/Main/Main.kicad_sch (KiCad schematic)
At the start: 53 parts, among them J1 USB_C_Receptacle_USB2.0, J10 Conn_01x06_Socket, J11 Conn_01x06_Socket, J12 Conn_01x06_Socket, J13 Conn_01x06_Socket, J14 Conn_01x06_Socket, J15 Conn_01x06_Socket, J16 Conn_01x06_Socket, J17 Conn_01x06_Socket, J2 Conn_01x06_Socket, J2 UJ32-C-V-G-TH-5-P24-TR, J21 Conn_01x04_Socket, J3 Conn_01x06_Socket, J4 Conn_01x06_Socket, J5 Conn_01x06_Socket, J6 Conn_01x06_Socket, J7 Conn_01x06_Socket, J8 Conn_01x06_Socket, J9 Conn_01x06_Socket, SW1 SW_Push, SW2 SW_Push, U1 RP2040, U3 Teensy4.0, U4 AE-BNO055-BO, U4 W25Q128JVS, U5 AZ1084-5.0, U6 AZ1084-3.3, Y1 Crystal_GND24

Commit message: KiCad変更
ごめんさい。溜めました
Parts:
- removed J2: UJ32-C-V-G-TH-5-P24-TR, UJ32-C-V-G-TH-5-P24-TR:SAMESKY_UJ32-C-V-G-TH-5-P24-TR, symbol UJ32-C-V-G-TH-5-P24-TR:UJ32-C-V-G-TH-5-P24-TR
- added C10, C11, C12, C7, C8, C9: C, Capacitor_SMD:C_0402_1005Metric, symbol Device:C
- added J14: UJ32-C-V-G-TH-5-P24-TR, Connector_USB:USB_C_Receptacle_GCT_USB4115-03-C, symbol UJ32-C-V-G-TH-5-P24-TR:UJ32-C-V-G-TH-5-P24-TR
- added J22, J23: Conn_01x06_Socket, Connector_JST:JST_XH_B6B-XH-A_1x06_P2.50mm_Vertical, symbol Connector:Conn_01x06_Socket
- BZ1: footprint (none) -> Buzzer_Beeper:Buzzer_Murata_PKLCS1212E
- C3: renamed from C4; footprint (none) -> Capacitor_SMD:C_1210_3225Metric_Pad1.33x2.70mm_HandSolder
- C4, C5: footprint (none) -> Capacitor_SMD:C_0402_1005Metric; LCSC (none) -> C1557
- C4: renamed from C3; footprint (none) -> Capacitor_SMD:C_1210_3225Metric_Pad1.33x2.70mm_HandSolder
- C5, C6: footprint (none) -> Capacitor_SMD:C_0402_1005Metric; LCSC (none) -> C1525
- J1: footprint (none) -> Connector_USB:USB_C_Receptacle_GCT_USB4105-xx-A_16P_TopMnt_Horizontal; LCSC (none) -> C136423
- J10: renamed from J4; footprint (none) -> Connector_PinHeader_2.54mm:PinHeader_1x06_P2.54mm_Horizontal
- J11: renamed from J8; footprint (none) -> Connector_PinHeader_2.54mm:PinHeader_1x06_P2.54mm_Horizontal
- J12, J2, J7: footprint (none) -> Connector_PinHeader_2.54mm:PinHeader_1x06_P2.54mm_Horizontal
- J13: renamed from J16; footprint (none) -> Connector_PinHeader_2.54mm:PinHeader_1x06_P2.54mm_Horizontal
- J15: renamed from J5; footprint (none) -> Connector_PinHeader_2.54mm:PinHeader_1x06_P2.54mm_Horizontal
- J16: renamed from J9; footprint (none) -> Connector_PinHeader_2.54mm:PinHeader_1x06_P2.54mm_Horizontal
- J17: renamed from J13; footprint (none) -> Connector_PinHeader_2.54mm:PinHeader_1x06_P2.54mm_Horizontal
- J18: renamed from J17; footprint (none) -> Connector_PinHeader_2.54mm:PinHeader_1x06_P2.54mm_Horizontal
- J2: footprint UJ32-C-V-G-TH-5-P24-TR:SAMESKY_UJ32-C-V-G-TH-5-P24-TR -> Connector_USB:USB_C_Receptacle_GCT_USB4115-03-C; LCSC (none) -> C5342428
- J21: footprint (none) -> Connector_JST:JST_XH_B4B-XH-A_1x04_P2.50mm_Vertical
- J3: renamed from J6; footprint (none) -> Connector_PinHeader_2.54mm:PinHeader_1x06_P2.54mm_Horizontal
- J4: renamed from J10; footprint (none) -> Connector_PinHeader_2.54mm:PinHeader_1x06_P2.54mm_Horizontal
- J5: renamed from J14; footprint (none) -> Connector_PinHeader_2.54mm:PinHeader_1x06_P2.54mm_Horizontal
- J6: renamed from J3; footprint (none) -> Connector_PinHeader_2.54mm:PinHeader_1x06_P2.54mm_Horizontal
- J8: renamed from J11; footprint (none) -> Connector_PinHeader_2.54mm:PinHeader_1x06_P2.54mm_Horizontal
- J9: renamed from J15; footprint (none) -> Connector_PinHeader_2.54mm:PinHeader_1x06_P2.54mm_Horizontal
- R4, R6: footprint (none) -> Resistor_SMD:R_0402_1005Metric; LCSC (none) -> C11702
- R5, R7: footprint (none) -> Resistor_SMD:R_0402_1005Metric; LCSC (none) -> C25100
- R8, R9: footprint (none) -> Resistor_SMD:R_0402_1005Metric; LCSC (none) -> C25905
- SW1, SW2: footprint (none) -> Button_Switch_THT:SW_Tactile_SPST_Angled_PTS645Vx31-2LFS
- SW3: renamed from SW1; footprint (none) -> Button_Switch_THT:SW_PUSH_6mm
- U1: LCSC (none) -> C2040
- U3: renamed from U5; footprint (none) -> Package_TO_SOT_SMD:TO-252-2
- U4: LCSC (none) -> C97521
- U4: renamed from U6; footprint (none) -> Package_TO_SOT_SMD:TO-252-2
- U5: renamed from U3; footprint (none) -> Teensy_Breakout:Teensy_Brakeout
- U6: renamed from U4; footprint (none) -> Package_DIP:CERDIP-8_W7.62mm_SideBrazed
- Y1: footprint (none) -> Crystal:Crystal_SMD_2520-4Pin_2.5x2.0mm; LCSC (none) -> C7294610
Connections:
- net +3V3 is gone; now on net +3.3V: J10.1 (Pin_1), J11.1 (Pin_1), J12.1 (Pin_1), J13.1 (Pin_1), J15.1 (Pin_1), J16.1 (Pin_1), J17.1 (Pin_1), J18.1 (Pin_1), J2.1 (Pin_1), J3.1 (Pin_1), J4.1 (Pin_1), J5.1 (Pin_1), J6.1 (Pin_1), J7.1 (Pin_1), J8.1 (Pin_1), J9.1 (Pin_1)
- net +12V: now also J14.A4 (VBUS), J14.A9 (VBUS), J14.B4 (VBUS), J14.B9 (VBUS)
- net +1V1: now also C7.1, C8.1
- net +3.3V: now also C10.1, C11.1, C12.1, C9.1, J22.1 (Pin_1), J22.3 (Pin_3), J23.1 (Pin_1), J23.3 (Pin_3)
- net 1: now also U1.17 (GPIO14); no longer U1.8 (GPIO6)
- net 10: now also U1.35 (GPIO23); no longer U1.18 (GPIO15)
- net 11: now also U1.36 (GPIO24); no longer U1.27 (GPIO16)
- net 12: now also U1.37 (GPIO25); no longer U1.28 (GPIO17)
- net 13: now also U1.38 (GPIO26_ADC0); no longer U1.29 (GPIO18)
- net 14: now also U1.39 (GPIO27_ADC1); no longer U1.30 (GPIO19)
- net 15: now also U1.40 (GPIO28_ADC2); no longer U1.31 (GPIO20)
- net 16: now also U1.41 (GPIO29_ADC3); no longer U1.32 (GPIO21)
- net 2: now also U1.18 (GPIO15); no longer U1.9 (GPIO7)
- net 3: now also U1.27 (GPIO16); no longer U1.11 (GPIO8)
- net 4: now also U1.28 (GPIO17); no longer U1.12 (GPIO9)
- net 5: now also U1.29 (GPIO18); no longer U1.13 (GPIO10)
- net 6: now also U1.30 (GPIO19); no longer U1.14 (GPIO11)
- net 7: now also U1.31 (GPIO20); no longer U1.15 (GPIO12)
- net 8: now also U1.32 (GPIO21); no longer U1.16 (GPIO13)
- net 9: now also U1.34 (GPIO22); no longer U1.17 (GPIO14)
- net FET1: now also J14.A6 (DP1)
- net FET2: now also J14.A7 (DN1)
- net FET3: now also J14.A5 (CC1)
- net GND: now also C10.2, C11.2, C12.2, C7.2, C8.2, C9.2, J14.A1 (GND), J14.A12 (GND), J14.B1 (GND), J14.B12 (GND), J14.SH1 (SHIELD), J14.SH2 (SHIELD), J14.SH3 (SHIELD), J14.SH4 (SHIELD), J22.2 (Pin_2), J23.2 (Pin_2)
- net LineRX: now also J14.B6 (DP2)
- net LineTX: now also J14.B7 (DN2)
- net Line_NeoPixel: now also J14.B8 (SBU2)
- net MDRX: now also J14.A3 (SSTXN1)
- net MDTX: now also J14.A2 (SSTXP1)
- net MouseRX: now also J14.B3 (SSTXN2)
- net MouseTX: now also J14.B5 (CC2)
- net ToF_RX: now also U1.15 (GPIO12); no longer U1.2 (GPIO0)
- net ToF_TX: now also U1.16 (GPIO13); no longer U1.3 (GPIO1)
- net Touch_B: now also J23.6 (Pin_6)
- net Touch_F: now also J22.6 (Pin_6)
- net UART_RX: now also J14.A8 (SBU1)
- net UART_TX: now also J14.A10 (SSRXN2)
- new net: J23.4 (Pin_4), J23.5 (Pin_5)
- new net: J22.4 (Pin_4), J22.5 (Pin_5)
