File: Project_Tsukuyomi (JapanOpen)/Hardware/KiCad/PSU/PSU.kicad_pcb (KiCad board)
At the start: 2 copper layers, 38 x 37.2 mm, 50 parts, among them J1 USB_C_Receptacle_USB2.0, J2 Conn_01x08_Socket, J3 Conn_01x08_Socket, J4 Conn_01x04_Socket, J5 Conn_01x02_Socket, J6 Conn_01x02_Socket, Q1 PMOS, SW1 SW_Push, SW2 SW_Push, U1 W25Q128JVS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

Commit message: KiCad変更
ごめんさい。溜めました
Parts:
- Y1: footprint Crystal:Crystal_SMD_2016-4Pin_2.0x1.6mm -> Crystal:Crystal_SMD_2520-4Pin_2.5x2.0mm
- moved C4 0.71 mm to (147.5, 96.0), turned to -90 degrees
- moved Y1 0.26 mm to (145.3, 95.8), turned to 0 degrees
Routing:
- net GND: track 15.2 -> 21.7 mm
- net Net-(U2-XIN): track 5.90 -> 9.89 mm
- net Net-(C5-Pad2): track 3.18 -> 2.34 mm
