File: Project_Tsukuyomi (JapanOpen)/Hardware/KiCad/Relay/Relay.kicad_sch (KiCad schematic)
At the start: 11 parts, among them J1 Conn_01x04_Socket, J2 UJ32-C-V-G-TH-5-P24-TR, J3 Conn_01x02_Socket, J4 Conn_01x02_Socket, J5 Conn_01x03_Socket, J6 Conn_01x05_Socket, J7 Conn_01x04_Socket, J8 Conn_01x08_Socket, J9 Conn_01x03_Socket

Commit message: KiCad変更
ごめんさい。溜めました
Parts:
- J1: renamed from J2; LCSC (none) -> C5342428
- J2: renamed from J6; footprint (none) -> Connector_JST:JST_XH_S5B-XH-A_1x05_P2.50mm_Horizontal
- J3, J4: footprint (none) -> Connector_AMASS:AMASS_XT30PW-M_1x02_P2.50mm_Horizontal
- J5: renamed from J9; footprint (none) -> Connector_JST:JST_XH_B3B-XH-A_1x03_P2.50mm_Vertical
- J6: renamed from J5; footprint (none) -> Connector_JST:JST_XH_B3B-XH-A_1x03_P2.50mm_Vertical
- J7: renamed from J1; footprint (none) -> Connector_PinSocket_2.54mm:PinSocket_1x04_P2.54mm_Horizontal
- J8: footprint (none) -> Connector_PinSocket_2.54mm:PinSocket_2x06_P2.54mm_Horizontal
- J9: renamed from J7; footprint (none) -> Connector_JST:JST_XH_B4B-XH-A_1x04_P2.50mm_Vertical
- U1, U2: footprint (none) -> ESC:ESC_20A
Connections:
- net +48V: now also J8.7 (Pin_7); no longer J8.8 (Pin_8)
- net BLDC2: now also J8.8 (Pin_8); no longer J8.7 (Pin_7)
- net FET1: now also J1.A6 (DP1); no longer J1.A10 (SSRXN2)
- net FET2: now also J1.A7 (DN1); no longer J1.A11 (SSRXP2)
- net FET3: now also J1.A5 (CC1); no longer J1.B3 (SSTXN2)
- net LineRX: now also J1.B6 (DP2); no longer J1.B10 (SSRXN1)
- net LineTX: now also J1.B7 (DN2); no longer J1.B11 (SSRXP1)
- net Line_NeoPixel: now also J1.B8 (SBU2); no longer J1.B2 (SSTXP2)
- net MDRX: now also J1.A3 (SSTXN1); no longer J1.A5 (CC1)
- net MDTX: now also J1.A2 (SSTXP1); no longer J1.A8 (SBU1)
- net MouseRX: now also J1.B3 (SSTXN2); no longer J1.B5 (CC2)
- net MouseTX: now also J1.B5 (CC2); no longer J1.B8 (SBU2)
- net UART_RX: now also J1.A8 (SBU1); no longer J1.A3 (SSTXN1)
- net UART_TX: now also J1.A10 (SSRXN2); no longer J1.A2 (SSTXP1)
