File: Project_Tsukuyomi (JapanOpen)/Hardware/KiCad/VoltageBooster/VoltageBooster.kicad_pcb (KiCad board)
At the start: 2 copper layers, 38 x 37.2 mm, 18 parts, among them J1 Conn_01x08_Socket, J2 Conn_01x08_Socket

Commit message: KiCad変更
ごめんさい。溜めました
Routing:
- net +48V: track 131.9 -> 141.9 mm, vias 0 -> 1
- net GND: vias 41 -> 32
Other:
- board text added: "+12v"
- board text added: "+48v"
- board text added: "GND"
- board text added: "VOLTAGE CHECK"
Changed lines of the file:
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@@
       (drillshape 0)
       (scaleselection 1)
-      (outputdirectory "untitled folder/")
+      (outputdirectory "VolageBooster/")
     )
   )
@@
   (gr_arc (start 151.35 113.745168) (mid 151.935787 112.330955) (end 153.35 111.745168)
     (stroke (width 0.2) (type solid)) (layer "Edge.Cuts"))
+  (gr_text "VOLTAGE CHECK" (at 138.32 118.56) (layer "F.SilkS")
+    (effects (font (size 1 1) (thickness 0.2) bold) (justify left bottom))
+  )
+  (gr_text "+12v" (at 142.3 116.91) (layer "F.SilkS")
+    (effects (font (size 0.8 0.8) (thickness 0.15) bold) (justify left bottom))
+  )
+  (gr_text "+48v" (at 146.39 116.95) (layer "F.SilkS")
+    (effects (font (size 0.8 0.8) (thickness 0.15) bold) (justify left bottom))
+  )
+  (gr_text "GND" (at 138.68 116.94) (layer "F.SilkS")
+    (effects (font (size 0.8 0.8) (thickness 0.15) bold) (justify left bottom))
+  )
   (segment (start 144.018 113.284) (end 147.828 109.474) (width 1) (layer "F.Cu") (net 1))
   (segment (start 147.686 107.046) (end 136.032 107.046) (width 3) (layer "F.Cu") (net 1))
@@
   (segment (start 147.828 107.188) (end 147.828 102.362) (width 2) (layer "B.Cu") (net 1))
   (segment (start 157.988 82.804) (end 159.512 82.804) (width 2) (layer "B.Cu") (net 1))
-  (via (at 149.88 98.54) (size 0.8) (drill 0.4) (layers "F.Cu" "B.Cu") (free) (net 2))
-  (via (at 150.114 109.59) (size 0.8) (drill 0.4) (layers "F.Cu" "B.Cu") (free) (net 2))
-  (via (at 150.622 114.554) (size 0.8) (drill 0.4) (layers "F.Cu" "B.Cu") (free) (net 2))
-  (via (at 155.37 109.76) (size 0.8) (drill 0.4) (layers "F.Cu" "B.Cu") (free) (net 2))
-  (via (at 145.542 109.728) (size 0.8) (drill 0.4) (layers "F.Cu" "B.Cu") (free) (net 2))
   (via (at 137.97 82.93) (size 0.8) (drill 0.4) (layers "F.Cu" "B.Cu") (free) (net 2))
   (via (at 143.53 83.23) (size 0.8) (drill 0.4) (layers "F.Cu" "B.Cu") (free) (net 2))
   (via (at 167.9 109.26) (size 0.8) (drill 0.4) (layers "F.Cu" "B.Cu") (free) (net 2))
   (via (at 167.77 102.19) (size 0.8) (drill 0.4) (layers "F.Cu" "B.Cu") (free) (net 2))
-  (via (at 151.56 99.78) (size 0.8) (drill 0.4) (layers "F.Cu" "B.Cu") (free) (net 2))
   (via (at 137.2 98.61) (size 0.8) (drill 0.4) (layers "F.Cu" "B.Cu") (free) (net 2))
   (via (at 170.67 110.02) (size 0.8) (drill 0.4) (layers "F.Cu" "B.Cu") (free) (net 2))
@@
   (via (at 141.9 109.59) (size 0.8) (drill 0.4) (layers "F.Cu" "B.Cu") (free) (net 2))
   (via (at 167.79 88.67) (size 0.8) (drill 0.4) (layers "F.Cu" "B.Cu") (free) (net 2))
-  (via (at 151.42 104.57) (size 0.8) (drill 0.4) (layers "F.Cu" "B.Cu") (free) (net 2))
   (via (at 169.31 111.98) (size 0.8) (drill 0.4) (layers "F.Cu" "B.Cu") (free) (net 2))
-  (via (at 145 99.32) (size 0.8) (drill 0.4) (layers "F.Cu" "B.Cu") (free) (net 2))
   (via (at 138.03 109.69) (size 0.8) (drill 0.4) (layers "F.Cu" "B.Cu") (free) (net 2))
   (via (at 164.44 90.71) (size 0.8) (drill 0.4) (layers "F.Cu" "B.Cu") (free) (net 2))
@@
   (via (at 168.63 83.71) (size 0.8) (drill 0.4) (layers "F.Cu" "B.Cu") (free) (net 2))
   (via (at 148.99 82.21) (size 0.8) (drill 0.4) (layers "F.Cu" "B.Cu") (free) (net 2))
-  (via (at 147.066 112.522) (size 0.8) (drill 0.4) (layers "F.Cu" "B.Cu") (free) (net 2))
   (via (at 164.46 82.14) (size 0.8) (drill 0.4) (layers "F.Cu" "B.Cu") (free) (net 2))
   (via (at 133.94 110.31) (size 0.8) (drill 0.4) (layers "F.Cu" "B.Cu") (free) (net 2))
@@
   (segment (start 150.647 90.429) (end 150.622 90.404) (width 1) (layer "F.Cu") (net 3))
   (segment (start 135.128 93.98) (end 135.763 94.615) (width 2) (layer "F.Cu") (net 3))
-  (segment (start 148.082 114.554) (end 148.082 113.792) (width 1) (layer "F.Cu") (net 3))
   (segment (start 135.128 92.71) (end 136.144 91.694) (width 2) (layer "F.Cu") (net 3))
   (segment (start 135.128 90.17) (end 152.979 90.17) (width 2) (layer "F.Cu") (net 3))
@@
   (segment (start 150.46 96.61) (end 150.46 90.566) (width 1) (layer "F.Cu") (net 3))
   (segment (start 152.979 90.17) (end 153.238 90.429) (width 2) (layer "F.Cu") (net 3))
-  (segment (start 152.71 109.164) (end 152.71 94.615) (width 1) (layer "F.Cu") (net 3))
   (segment (start 150.46 90.566) (end 150.622 90.404) (width 1) (layer "F.Cu") (net 3))
   (segment (start 135.487138 95.25) (end 136.757138 96.52) (width 2) (layer "F.Cu") (net 3))
   (segment (start 135.128 95.25) (end 135.128 93.98) (width 2) (layer "F.Cu") (net 3))
-  (segment (start 148.082 113.792) (end 152.71 109.164) (width 1) (layer "F.Cu") (net 3))
   (segment (start 135.128 93.98) (end 135.128 90.17) (width 2) (layer "F.Cu") (net 3))
+  (via (at 148.11 114.57) (size 0.8) (drill 0.4) (layers "F.Cu" "B.Cu") (net 3))
+  (segment (start 155.43 111.19) (end 157.225 109.395) (width 0.25) (layer "B.Cu") (net 3))
+  (segment (start 152.898167 111.19) (end 155.43 111.19) (width 0.25) (layer "B.Cu") (net 3))
+  (segment (start 149.518167 114.57) (end 152.898167 111.19) (width 0.25) (layer "B.Cu") (net 3))
+  (segment (start 157.225 109.395) (end 157.225 94.416) (width 0.25) (layer "B.Cu") (net 3))
+  (segment (start 148.11 114.57) (end 149.518167 114.57) (width 0.25) (layer "B.Cu") (net 3))
+  (segment (start 157.225 94.416) (end 153.238 90.429) (width 0.25) (layer "B.Cu") (net 3))
   (segment (start 157.226 92.71) (end 159.004 92.71) (width 2) (layer "F.Cu") (net 4))
   (segment (start 156.21 92.71) (end 157.226 92.71) (width 2) (layer "F.Cu") (net 4))
@@
       )
     )
+  )
+  (zone (net 0) (net_name "") (layers "F&B.Cu") (hatch edge 0.5)
+    (connect_pads (clearance 0))
+    (min_thickness 0.25) (filled_areas_thickness no)
+    (keepout (tracks not_allowed) (vias not_allowed) (pads not_allowed) (copperpour not_allowed) (footprints allowed))
+    (fill (thermal_gap 0.5) (thermal_bridge_width 0.5))
+    (polygon
+      (pts
+        (xy 144.02 98.51)
+        (xy 144.01 111.26)
+        (xy 156.73 111.26)
+        (xy 156.73 98.54)
+      )
+    )
