File: Project_Tsukuyomi (JapanOpen)/Hardware/KiCad/IO/IO.kicad_pcb (KiCad board)
At the start: 2 copper layers, 140 x 140 mm, 87 parts, among them J1 Conn_01x14_Socket, J2 Conn_01x04_Socket, J3 Conn_01x04_Socket, J4 UJ32-C-V-G-TH-5-P24-TR, J5 Conn_01x07_Socket, U1 AZ1084-3.3, U2 AZ1084-5.0, U3 TWE-L-WX

Commit message: 溜まった変更大放出
Parts:
- added J1: Conn_01x01_Socket, TestPoint:TestPoint_Pad_D1.0mm, B.Cu at (143.4, 66.5)
- added J10: Conn_01x01_Socket, TestPoint:TestPoint_Pad_D1.0mm, B.Cu at (146.9, 64.8)
- added J12: Conn_01x01_Socket, TestPoint:TestPoint_Pad_D1.0mm, B.Cu at (145.2, 68.3)
- added J13: Conn_01x01_Socket, TestPoint:TestPoint_Pad_D1.0mm, B.Cu at (143.4, 70.0)
- added J14: Conn_01x01_Socket, TestPoint:TestPoint_Pad_D1.0mm, B.Cu at (143.4, 68.3)
- added J15: Conn_01x01_Socket, TestPoint:TestPoint_Pad_D1.0mm, B.Cu at (141.7, 68.3)
- added J16: Conn_01x01_Socket, TestPoint:TestPoint_Pad_D1.0mm, B.Cu at (139.9, 68.3)
- added J17: Conn_01x01_Socket, TestPoint:TestPoint_Pad_D1.0mm, B.Cu at (141.6, 70.1)
- added J18: Conn_01x01_Socket, TestPoint:TestPoint_Pad_D1.0mm, B.Cu at (145.2, 70.0)
- added J19: Conn_01x01_Socket, TestPoint:TestPoint_Pad_D1.0mm, B.Cu at (146.9, 68.3)
- added J2: Conn_01x01_Socket, TestPoint:TestPoint_Pad_D1.0mm, B.Cu at (141.7, 66.5)
- added J20: Conn_01x01_Socket, TestPoint:TestPoint_Pad_D1.0mm, B.Cu at (146.9, 70.0)
- added J21: Conn_01x01_Socket, TestPoint:TestPoint_Pad_D1.0mm, B.Cu at (148.7, 70.0)
- added J22: Conn_01x01_Socket, TestPoint:TestPoint_Pad_D1.0mm, B.Cu at (146.9, 66.5)
- added J3: Conn_01x01_Socket, TestPoint:TestPoint_Pad_D1.0mm, B.Cu at (141.7, 64.7)
- added J5: Conn_01x01_Socket, TestPoint:TestPoint_Pad_D1.0mm, B.Cu at (145.2, 66.5)
- added J6: Conn_01x01_Socket, TestPoint:TestPoint_Pad_D1.0mm, B.Cu at (145.2, 64.7)
- added J7: Conn_01x01_Socket, TestPoint:TestPoint_Pad_D1.0mm, B.Cu at (139.9, 66.5)
- added J8: Conn_01x01_Socket, TestPoint:TestPoint_Pad_D1.0mm, B.Cu at (138.2, 66.5)
- added J9: Conn_01x01_Socket, TestPoint:TestPoint_Pad_D1.0mm, B.Cu at (139.9, 64.7)
- J4: value UJ32-C-V-G-TH-5-P24-TR -> Conn_01x01_Socket; footprint Connector_USB:USB_C_Receptacle_GCT_USB4115-03-C -> TestPoint:TestPoint_Pad_D1.0mm
- moved J4 1.53 mm to (143.4, 64.7), turned to 0 degrees
Routing:
- net +12V: track 134.6 -> 127.7 mm, vias 4 -> 2
- net /PWM: track 53.9 -> 60.0 mm
- net /SD＿SCK: track 65.2 -> 61.0 mm
- net +5V: track 600.8 -> 597.0 mm
- net /T_CS: track 87.8 -> 84.3 mm
- net /SCK: track 81.4 -> 78.5 mm
- net /RXD: track 58.3 -> 55.7 mm
- net /SD＿CS: track 57.2 -> 59.7 mm
- net /RESET: track 63.1 -> 60.6 mm
- net /START: track 99.9 -> 97.4 mm
- net /SD＿MISO: track 61.1 -> 58.9 mm
- net GND: track 2.90 -> 0.90 mm, vias 139 -> 135
- net /DC: track 66.3 -> 64.7 mm
- net /MISO: track 99.7 -> 98.4 mm
- net /MOSI: track 92.2 -> 91.1 mm
