File: Project_Tsukuyomi (JapanOpen)/Hardware/KiCad/IO/IO.kicad_sch (KiCad schematic)
At the start: 76 parts, among them J1 Conn_01x04_Socket, J2 Conn_01x14_Socket, J2 UJ32-C-V-G-TH-5-P24-TR, J3 Conn_01x04_Socket, J5 Conn_01x07_Socket, U1 TWE-L-WX, U2 AZ1084-3.3, U3 AZ1084-5.0

Commit message: KiCad変更
ごめんさい。溜めました
Parts:
- C1, C3: footprint (none) -> Capacitor_SMD:C_1210_3225Metric_Pad1.33x2.70mm_HandSolder
- C2, C4: footprint (none) -> Capacitor_THT:C_Disc_D3.0mm_W1.6mm_P2.50mm
- D1, D10, D11, D12, D13, D14, D15, D16, D17, D18, D19, D2, D20, D21, D22, D23, D24, D25, D26, D27, D28, D29, D3, D30, D31, D32, D33, D34, D35, D36, D37, D38, D39, D4, D40, D41, D42, D43, D44, D45, D46, D47, D48, D49, D5, D50, D51, D52, D53, D54, D55, D56, D57, D58, D59, D6, D60, D61, D62, D63, D64, D7, D8, D9: footprint LED_SMD:LED_WS2812B_PLCC4_5.0x5.0mm_P3.2mm -> LED_SMD:LED_WS2812B-2020_PLCC4_2.0x2.0mm
- J1: renamed from J2; footprint (none) -> Connector_PinHeader_2.54mm:PinHeader_1x14_P2.54mm_Vertical
- J2: renamed from J1; footprint (none) -> Connector_JST:JST_XH_B4B-XH-A_1x04_P2.50mm_Vertical
- J2: footprint UJ32-C-V-G-TH-5-P24-TR:SAMESKY_UJ32-C-V-G-TH-5-P24-TR -> Connector_USB:USB_C_Receptacle_GCT_USB4115-03-C
- J3: footprint (none) -> Connector_PinHeader_2.54mm:PinHeader_1x04_P2.54mm_Vertical
- J5: footprint (none) -> Connector_PinHeader_2.54mm:PinHeader_1x07_P2.54mm_Vertical
- U1: renamed from U2; footprint (none) -> Package_TO_SOT_SMD:TO-252-2
- U2: renamed from U3; footprint (none) -> Package_TO_SOT_SMD:TO-252-2
- renumbered U1 to U3

Commit message: 溜まった変更大放出
Parts:
- added J16: DX07P024MJ1R1500, DX07P024MJ1R1500:JAE_DX07P024MJ1R1500, symbol DX07P024MJ1R150:DX07P024MJ1R1500
Connections:
- net +12V: now also J16.A4 (A_VBUS), J16.A9 (A_VBUS), J16.B4 (B_VBUS), J16.B9 (B_VBUS)
- net CS: now also J16.B5 (CC2)
- net DC: now also J16.B2 (TX2+)
- net GND: now also J16.A1 (GNDA), J16.A12 (GNDA), J16.B1 (GNDB), J16.B12 (GNDB), J16.S3 (SHIELD), J16.S4 (SHIELD), J16.S5 (SHIELD), J16.S6 (SHIELD)
- net MISO: now also J16.A5 (CC1)
- net MOSI: now also J16.A8 (SBU1)
- net PWM: now also J16.B6 (DB+)
- net RESET: now also J16.B3 (TX2-)
- net RXD: now also J16.A7 (DA-)
- net SCK: now also J16.A11 (RX2+)
- net SD＿CS: now also J16.A2 (TX1+)
- net SD＿MISO: now also J16.B11 (RX1+)
- net SD＿MOSI: now also J16.A3 (TX1-)
- net SD＿SCK: now also J16.B10 (RX1-)
- net START: now also J16.B8 (SBU2)
- net TXD: now also J16.A6 (DA+)
- net T_CS: now also J16.A10 (RX2-)
- no-connect marks 4 -> 5
